File: pi-shield/pi-shield.brd (EAGLE design)
At the start: 133.3 x 144.4 mm, 19 parts, among them J1 PINHD-3X4

Commit message: Calibration Windows
I've opened up windows above POT1-3 and U9, pin 10. The windows allow access to the pots and U9 for initial calibration of the PI controller.

DSB
Routing:
- net N$23: track 139.8 -> 129.0 mm
- net +12V: track 138.8 -> 129.1 mm
- net N$22: track 139.1 -> 130.9 mm
- net N$15: track 58.6 -> 60.5 mm
- net N$13: track 52.8 -> 54.0 mm
- net N$48: track 49.1 -> 48.3 mm
- net N$49: track 56.3 -> 55.5 mm
Other:
- outline, holes or cut-outs redrawn
